File: pcb files/usb hub.kicad_pcb (KiCad board)
At the start: 2 copper layers, 62.5 x 37.5 mm, 11 parts, among them J1 USB_C_Receptacle_USB2.0_16P, U1 SL2.1A

Commit message: added pcb files
Parts:
- added G***: LOGO, LOGO, F.Cu at (149.0, 87.5)
- added G***: LOGO, LOGO, F.Cu at (122.0, 79.0)
Routing:
- net GND: track 300.8 -> 370.1 mm, vias 2 -> 11
- net Net-(U1-DP3): track 53.2 -> 73.5 mm, vias 0 -> 3
- net +5V: track 155.0 -> 161.7 mm, vias 0 -> 2
- net Net-(U1-DM3): track 22.4 -> 25.2 mm, vias 0 -> 3
Other:
- board text added: "2.0"
- board text added: "USB-HUB"
